File: Placa/fondo/fondo.kicad_pcb (KiCad board)
At the start: 2 copper layers, 34 parts, among them J1 Conn_01x08, J1 L298N, J2 Encoder, J3 Calibre, J4 Fotoeléctrico, J5 Conn_01x04, J7 Digitales, Q1 2N2222A, Q2 2N2222A, SW5 Enter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

Commit message: Diseño de placa
Parts:
- removed J1: L298N, TerminalBlock_TE-Connectivity:TerminalBlock_TE_282834-6_1x06_P2.54mm_Horizontal
- removed J1: Conn_01x08, TerminalBlock_Phoenix:TerminalBlock_Phoenix_MPT-0,5-8-2.54_1x08_P2.54mm_Horizontal
- removed J2: Encoder, TerminalBlock_TE-Connectivity:TerminalBlock_TE_282834-4_1x04_P2.54mm_Horizontal
- removed J3: Calibre, TerminalBlock_TE-Connectivity:TerminalBlock_TE_282834-4_1x04_P2.54mm_Horizontal
- removed SW5: Enter, Button_Switch_THT:SW_PUSH_6mm_H8mm
- removed SW6: ESC, Button_Switch_THT:SW_PUSH_6mm_H8mm
- added H1: MountingHole_Pad, MountingHole:MountingHole_3.2mm_M3_DIN965_Pad, F.Cu at (111.8, 53.2)
- added H2: MountingHole_Pad, MountingHole:MountingHole_3.2mm_M3_DIN965_Pad, F.Cu at (177.8, 53.2)
- added H3: MountingHole_Pad, MountingHole:MountingHole_3.2mm_M3_DIN965_Pad, F.Cu at (111.8, 134.5)
- added H4: MountingHole_Pad, MountingHole:MountingHole_3.2mm_M3_DIN965_Pad, F.Cu at (177.8, 134.5)
- added J0: Conn_01x03, TerminalBlock:TerminalBlock_bornier-3_P5.08mm, F.Cu at (174.0, 115.4)
- added J1A1: Conn_01x05, TerminalBlock_TE-Connectivity:TerminalBlock_TE_282834-5_1x05_P2.54mm_Horizontal, F.Cu at (116.8, 120.5)
- added J1B1: Conn_01x05, TerminalBlock_TE-Connectivity:TerminalBlock_TE_282834-5_1x05_P2.54mm_Horizontal, F.Cu at (116.8, 105.3)
- added J1C1: Conn_01x05, TerminalBlock_TE-Connectivity:TerminalBlock_TE_282834-5_1x05_P2.54mm_Horizontal, F.Cu at (116.8, 90.0)
- added J1D1: Conn_01x04, TerminalBlock_TE-Connectivity:TerminalBlock_TE_282834-4_1x04_P2.54mm_Horizontal, F.Cu at (116.8, 74.8)
- added J2A1: Conn_01x03, TerminalBlock_TE-Connectivity:TerminalBlock_TE_282834-3_1x03_P2.54mm_Horizontal, F.Cu at (120.7, 54.5)
- added J2B1: Conn_01x04, TerminalBlock_TE-Connectivity:TerminalBlock_TE_282834-4_1x04_P2.54mm_Horizontal, F.Cu at (130.2, 54.5)
- added J2C1: Conn_01x05, TerminalBlock_TE-Connectivity:TerminalBlock_TE_282834-5_1x05_P2.54mm_Horizontal, F.Cu at (142.2, 54.5)
- added J2D1: Conn_01x03, TerminalBlock_TE-Connectivity:TerminalBlock_TE_282834-3_1x03_P2.54mm_Horizontal, F.Cu at (156.8, 54.5)
- added J3A1: Conn_01x03, TerminalBlock:TerminalBlock_bornier-3_P5.08mm, F.Cu at (174.0, 98.9)
- added J3B1: Conn_01x03, TerminalBlock_TE-Connectivity:TerminalBlock_TE_282834-3_1x03_P2.54mm_Horizontal, F.Cu at (174.0, 83.8)
- added J6: Fotoeléctrico, TerminalBlock_TE-Connectivity:TerminalBlock_TE_282834-4_1x04_P2.54mm_Horizontal, F.Cu at (137.2, 130.7)
- J4: value Fotoeléctrico -> Encoder
- J5: value Conn_01x04 -> Calibre
- moved J4 146.2 mm to (124.5, 130.7), turned to 180 degrees
- moved J5 107.6 mm to (149.9, 130.7), turned to 180 degrees
- moved R17 83.8 mm to (156.2, 135.7), turned to 90 degrees
- moved R1 78.3 mm to (128.3, 65.9)
- moved R2 78.3 mm to (128.3, 71.0)
- moved R3 78.3 mm to (128.3, 76.1)
- moved R4 78.3 mm to (128.3, 81.1)
- moved R20 78.3 mm to (166.4, 129.4), turned to 90 degrees
- moved U1 75.8 mm to (142.2, 63.4)
- moved R5 73.3 mm to (153.7, 65.9)
- moved R6 73.3 mm to (153.7, 71.0)
- moved R7 73.3 mm to (153.7, 76.1)
- moved R8 73.3 mm to (153.7, 81.1)
- moved R19 71.3 mm to (171.4, 135.7), turned to 90 degrees
- moved R15 68.1 mm to (138.4, 116.7), turned to 180 degrees
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Connections:
- J4 pad 1: +24V -> +5V
- J4 pad 2: +24V -> GND
- J4 pad 3: GND -> FASEA
- J4 pad 4: FOTO24V -> FASEB
- J5 pad 1: +5V -> +1V5
- J5 pad 3: SDA -> CLK1V5
- J5 pad 4: SCL -> DATOS1V5
Routing:
- net +5V: track 0.00 -> 231.1 mm
- net +24V: track 0.00 -> 194.6 mm, vias 0 -> 1
- net IN3: track 0.00 -> 151.8 mm, vias 0 -> 2
- net IN4: track 0.00 -> 149.8 mm, vias 0 -> 3
- net ENB: track 0.00 -> 146.7 mm, vias 0 -> 1
- net DATOS5V: track 0.00 -> 145.9 mm, vias 0 -> 1
- net CLK5V: track 0.00 -> 133.0 mm, vias 0 -> 2
- net FOTO24V: track 0.00 -> 122.2 mm, vias 0 -> 2
- net MICRO5V: track 0.00 -> 90.2 mm, vias 0 -> 3
- net SCL: track 0.00 -> 83.6 mm, vias 0 -> 1
- net SDA: track 0.00 -> 79.3 mm
- net UP: track 0.00 -> 76.3 mm
- net AVANCE: track 0.00 -> 72.8 mm
- net RETROCESO: track 0.00 -> 72.6 mm, vias 0 -> 3
- net DOWN: track 0.00 -> 72.5 mm
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- added copper zone on B.Cu, net GND
- added copper zone on F.Cu, net GND
Other:
- board outline added: 73.2 x 88.7 mm

Commit message: Finalización placas
Parts:
- removed J2C1: Conn_01x05, TerminalBlock_TE-Connectivity:TerminalBlock_TE_282834-5_1x05_P2.54mm_Horizontal
- added D1: LED, LED_THT:LED_D3.0mm, F.Cu at (158.4, 100.3)
- added D2: LED, LED_THT:LED_D3.0mm, F.Cu at (164.7, 100.3)
- added D3: LED, LED_THT:LED_D3.0mm, F.Cu at (158.4, 106.7)
- added D4: LED, LED_THT:LED_D3.0mm, F.Cu at (164.7, 106.7)
- added J7: Tapa, TerminalBlock_TE-Connectivity:TerminalBlock_TE_282834-4_1x04_P2.54mm_Horizontal, F.Cu at (142.2, 54.5)
- J0: value Conn_01x03 -> Alimentación
- J1: renamed from J1A1; value Conn_01x05 -> Arduino
- J10: renamed from J3A1; value Conn_01x03 -> L298N
- J11: renamed from J3B1; value Conn_01x03 -> L298N
- J2: renamed from J1B1; value Conn_01x05 -> Arduino
- J3: renamed from J1C1; value Conn_01x05 -> Arduino
- J4: renamed from J1D1; value Conn_01x04 -> Arduino
- J5: renamed from J2A1; value Conn_01x03 -> Tapa
- J6: renamed from J2B1; value Conn_01x04 -> Tapa
- J8: renamed from J2D1; value Conn_01x03 -> Tapa
- R1, R10, R2, R3, R4, R9: value 2k -> 8k2
- R11, R12: value 2k -> 4k7
- R13, R14: value 2k -> 2k6
- R5, R6, R7, R8: value 2k -> 1k
- U1, U2: footprint Package_DIP:DIP-16_W7.62mm -> Package_DIP:DIP-16_W10.16mm
- moved R13 2.54 mm to (156.2, 88.8)
- moved R14 2.54 mm to (156.2, 93.8)
- moved R5 2.54 mm to (156.2, 65.9)
- moved R6 2.54 mm to (156.2, 71.0)
- moved R7 2.54 mm to (156.2, 76.1)
- moved R8 2.54 mm to (156.2, 81.1)
- moved J8 2.49 mm to (154.4, 54.5)
- moved R15 1.41 mm to (138.4, 118.1)
- moved U3 1.28 mm to (143.5, 111.8)
- renumbered J4 to J12, J5 to J13, J6 to J14, J7 to J9
Connections:
- R5 pad 2: GND -> Net-(R5-Pad2)
- R6 pad 2: GND -> Net-(R6-Pad2)
- R7 pad 2: GND -> Net-(R7-Pad2)
- R8 pad 2: GND -> Net-(R8-Pad2)
- U2 pad 5: EMER5V -> EMER24V
- U2 pad 7: EMER5V -> EMER24V
Routing:
- net ENB: track 146.7 -> 92.4 mm, vias 1 -> 0
- net EMER24V: track 65.2 -> 111.3 mm, vias 0 -> 1
- net Net-(R5-Pad2): track 0.00 -> 38.8 mm
- net Net-(R7-Pad2): track 0.00 -> 35.0 mm
- net Net-(R6-Pad2): track 0.00 -> 32.0 mm
- net Net-(R8-Pad2): track 0.00 -> 29.7 mm
- net +5V: track 231.1 -> 255.4 mm
- net +24V: track 194.6 -> 209.2 mm
- net EMER5V: track 57.9 -> 44.1 mm
- net RETROCESO: track 72.6 -> 82.6 mm
- net SCL: track 83.6 -> 92.5 mm, vias 1 -> 0
- net MICRO24V: track 63.0 -> 68.6 mm
- net IN3: track 151.8 -> 148.2 mm
- net LR5V: track 49.7 -> 53.4 mm
- net FOTO24V: track 122.2 -> 125.4 mm
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Other:
- board text added: "1V5"
- board text added: "24V"
- board text added: "2N2222A"
- board text added: "39k"
- board text added: "5V"
- board text added: "AV"
- board text added: "Arduino"
- board text added: "Autor: Antonio Pérez García Trabajo Fin de Grado. 2022"
- board text added: "CLK 1V5"
- board text added: "CLK5"
- board text added: "COM"
- board text added: "DAT 1V5"
- board text added: "DAT5"
- board text added: "DOWN"
- board text added: "EM24"
- board text added: "EM5"
- board text added: "EMER"
- board text added: "ENB"
- board text added: "ENTER"
- board text added: "ESC"
- board text added: "FASEA"
- board text added: "FASEB"
- board text added: "FE24"
- board text added: "FE5"
- board text added: "FOTO"
- board text added: "GND"
- board text added: "IN3"
- board text added: "IN4"
- board text added: "L298N"
- board text added: "LR"
- board text added: "LR24"
- board text added: "LR5"
- board text added: "MC24"
- board text added: "MC5"
- board text added: "MICRO"
- board text added: "RETR"
- board text added: "SCL"
- board text added: "SDA"
- board text added: "TL082"
- board text added: "TLP-621-4GRG"
- board text added: "Tapa"
- board text added: "UP"
