File: Placa/fondo/fondo.kicad_sch (KiCad schematic)
At the start: 39 parts, among them J1 L298N, J2 Encoder, J24 Digitales, J3 Calibre, J4 Fotoeléctrico, J5 Conn_01x04, J6 Arduino, J7 Tapa, Q1 2N2222A, Q2 2N2222A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

Commit message: Diseño de placa
Parts:
- removed J1: L298N, TerminalBlock_TE-Connectivity:TerminalBlock_TE_282834-6_1x06_P2.54mm_Horizontal, symbol Connector_Generic:Conn_01x06
- removed J5: Conn_01x04, TerminalBlock_TE-Connectivity:TerminalBlock_TE_282834-4_1x04_P2.54mm_Horizontal, symbol Connector_Generic:Conn_01x04
- removed J6: Arduino, symbol Connector_Generic:Conn_01x19
- removed J7: Tapa, symbol Connector_Generic:Conn_01x15
- removed SW1: Botón Selección, symbol Switch:SW_DPDT_x2
- removed SW2: LR, symbol Switch:SW_DIP_x01
- removed SW3: MICRO, symbol Switch:SW_DIP_x01
- removed SW4: EMERGENCIA, symbol Switch:SW_DIP_x01
- removed SW5: Enter, TerminalBlock_TE-Connectivity:TerminalBlock_TE_282834-2_1x02_P2.54mm_Horizontal, symbol Switch:SW_Push
- removed SW6: ESC, TerminalBlock_TE-Connectivity:TerminalBlock_TE_282834-2_1x02_P2.54mm_Horizontal, symbol Switch:SW_Push
- added H1, H2, H3, H4: MountingHole_Pad, MountingHole:MountingHole_3.2mm_M3_DIN965_Pad, symbol Mechanical:MountingHole_Pad
- added J0, J3A1: Conn_01x03, TerminalBlock:TerminalBlock_bornier-3_P5.08mm, symbol Connector_Generic:Conn_01x03
- added J1A1, J1B1, J1C1, J2C1: Conn_01x05, TerminalBlock_TE-Connectivity:TerminalBlock_TE_282834-5_1x05_P2.54mm_Horizontal, symbol Connector_Generic:Conn_01x05
- added J1D1, J2B1: Conn_01x04, TerminalBlock_TE-Connectivity:TerminalBlock_TE_282834-4_1x04_P2.54mm_Horizontal, symbol Connector_Generic:Conn_01x04
- added J2A1, J2D1, J3B1: Conn_01x03, TerminalBlock_TE-Connectivity:TerminalBlock_TE_282834-3_1x03_P2.54mm_Horizontal, symbol Connector_Generic:Conn_01x03
- renumbered J2 to J4, J3 to J5, J4 to J6, J24 to J7
Connections:
- net +24V: now also J0.3 (Pin_3), J2A1.3 (Pin_3), J3A1.3 (Pin_3)
- net +5V: now also J0.2 (Pin_2), J1A1.1 (Pin_1), J2A1.2 (Pin_2), J3A1.1 (Pin_1)
- net AVANCE: now also J2C1.3 (Pin_3)
- net CLK5V: now also J1D1.1 (Pin_1)
- net DATOS5V: now also J1D1.2 (Pin_2)
- net DOWN: now also J1C1.1 (Pin_1), J2C1.2 (Pin_2)
- net EMER24V: now also J2D1.3 (Pin_3)
- net EMER5V: now also J1C1.4 (Pin_4)
- net ENB: now also J1A1.3 (Pin_3), J2C1.4 (Pin_4), J3B1.3 (Pin_3)
- net ENTER: now also J1B1.4 (Pin_4), J2B1.1 (Pin_1)
- net ESC: now also J1B1.3 (Pin_3), J2B1.2 (Pin_2)
- net FASEA: now also J1A1.5 (Pin_5)
- net FASEB: now also J1A1.4 (Pin_4)
- net FOTO5V: now also J1C1.5 (Pin_5)
- net GND: now also H1.1, H2.1, H3.1, H4.1, J0.1 (Pin_1), J1A1.2 (Pin_2), J2A1.1 (Pin_1), J3A1.2 (Pin_2)
- net IN3: now also J1D1.3 (Pin_3), J3B1.1 (Pin_1)
- net IN4: now also J1D1.4 (Pin_4), J3B1.2 (Pin_2)
- net LR24V: now also J2D1.1 (Pin_1)
- net LR5V: now also J1C1.2 (Pin_2)
- net MICRO24V: now also J2D1.2 (Pin_2)
- net MICRO5V: now also J1C1.3 (Pin_3)
- net RETROCESO: now also J2C1.5 (Pin_5)
- net SCL: now also J1B1.2 (Pin_2), J2B1.4 (Pin_4)
- net SDA: now also J1B1.1 (Pin_1), J2B1.3 (Pin_3)
- net UP: now also J1B1.5 (Pin_5), J2C1.1 (Pin_1)
Other:
- note added: "Agujeros de montaje"
- note added: "Alimentación sistema"
- note removed: "Botones enter y escape"
- note removed: "Botón de selección"
- note removed: "Conexiones LCD"
- note removed: "Switches de estado"
- moved on the sheet: J4, J5, J6, J7

Commit message: Finalización placas
Parts:
- removed J2C1: Conn_01x05, TerminalBlock_TE-Connectivity:TerminalBlock_TE_282834-5_1x05_P2.54mm_Horizontal, symbol Connector_Generic:Conn_01x05
- added D1, D2, D3, D4: LED, LED_THT:LED_D3.0mm, symbol Device:LED
- added J7: Tapa, TerminalBlock_TE-Connectivity:TerminalBlock_TE_282834-4_1x04_P2.54mm_Horizontal, symbol Connector_Generic:Conn_01x04
- J0: value Conn_01x03 -> Alimentación
- J1: renamed from J1A1; value Conn_01x05 -> Arduino
- J10: renamed from J3A1; value Conn_01x03 -> L298N
- J11: renamed from J3B1; value Conn_01x03 -> L298N
- J2: renamed from J1B1; value Conn_01x05 -> Arduino
- J3: renamed from J1C1; value Conn_01x05 -> Arduino
- J4: renamed from J1D1; value Conn_01x04 -> Arduino
- J5: renamed from J2A1; value Conn_01x03 -> Tapa
- J6: renamed from J2B1; value Conn_01x04 -> Tapa
- J8: renamed from J2D1; value Conn_01x03 -> Tapa
- R1, R10, R2, R3, R4, R9: value 2k -> 8k2
- R11, R12: value 2k -> 4k7
- R13, R14: value 2k -> 2k6
- R5, R6, R7, R8: value 2k -> 1k
- U1, U2: footprint Package_DIP:DIP-16_W7.62mm -> Package_DIP:DIP-16_W10.16mm
- renumbered J4 to J12, J5 to J13, J6 to J14, J7 to J9
Connections:
- net AVANCE: now also J7.3 (Pin_3)
- net DOWN: now also J7.2 (Pin_2)
- net EMER24V: now also U2.5, U2.7
- net EMER5V: no longer U2.5, U2.7
- net GND: now also D1.1 (K), D2.1 (K), D3.1 (K), D4.1 (K); no longer R5.2, R6.2, R7.2, R8.2
- net RETROCESO: now also J7.4 (Pin_4)
- net UP: now also J7.1 (Pin_1)
- new net: D3.2 (A), R7.2
- new net: D2.2 (A), R6.2
- new net: D1.2 (A), R5.2
- new net: D4.2 (A), R8.2
