File: Placa/fondo/fondo.kicad_sch (KiCad schematic)
At the start: 48 parts, among them J0 Alimentación, J1 Arduino, J10 L298N, J11 L298N, J12 Encoder, J13 Calibre, J14 Fotoeléctrico, J2 Arduino, J3 Arduino, J4 Arduino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

Commit message: FINAL
Other:
- title: (none) -> Esquemático placa de la base
Changed lines of the file:
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@@
 (kicad_sch (version 20211123) (generator eeschema)
   (paper "A4")
+  (title_block
+    (title "Esquemático placa de la base")
+    (date "2022-02-25")
+  )
   (junction (at 255.27 35.56) (diameter 0) (color 0 0 0 0)
   )
