File: Placa/tapa/tapa.kicad_pcb (KiCad board)
At the start: 2 copper layers, 89.4 x 37.5 mm, 15 parts, among them J1 Conn_01x03, J2 Conn_01x04, J3 Conn_01x05, J4 Conn_01x03, J5 Conn_01x04, SW1 Enter, SW2 ESC, SW3 Botón Selección, SW4 LR, SW5 MICRO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

Commit message: Finalización placas
Parts:
- J3: value Conn_01x05 -> Conn_01x04; footprint TerminalBlock_TE-Connectivity:TerminalBlock_TE_282834-5_1x05_P2.54mm_Horizontal -> TerminalBlock_TE-Connectivity:TerminalBlock_TE_282834-4_1x04_P2.54mm_Horizontal
- J5: value Conn_01x04 -> LCD
- SW1, SW2: moved to B.Cu
- moved SW2 66.4 mm to (153.1, 67.6), turned to 180 degrees
- moved J5 13.0 mm to (86.4, 59.7)
- moved SW3 11.7 mm to (100.3, 59.7)
- moved SW4 10.5 mm to (119.4, 59.7)
- moved SW5 10.5 mm to (127.0, 59.7)
- moved SW6 10.5 mm to (134.6, 59.7)
- moved SW1 8.19 mm to (76.9, 67.6), turned to 180 degrees
- moved J2 2.29 mm to (100.3, 80.6)
- moved J4 2.29 mm to (128.3, 80.6)
- moved J1 1.91 mm to (88.9, 80.7)
- moved J3 1.91 mm to (114.3, 80.6)
Connections:
- J1 pad 1: +5V -> GND
- J1 pad 2: GND -> +5V
- J3 pad 4: MICRO5V_B -> RETROCESO
- SW3 pad 5: MICRO5V_B -> MICRO24V
Routing:
- net ESC: track 25.0 -> 58.0 mm
- net MICRO24V: track 18.6 -> 47.3 mm
- net MICRO5V_B: track 16.5 -> 0.00 mm
- net SDA: track 16.5 -> 26.7 mm
- net SCL: track 16.5 -> 26.7 mm
- net UP: track 16.5 -> 25.7 mm
- net DOWN: track 16.5 -> 25.7 mm
- net AVANCE: track 16.5 -> 25.7 mm
- net LR24V: track 16.5 -> 24.6 mm
- net RETROCESO: track 16.5 -> 24.6 mm
- net +24V: track 76.1 -> 80.5 mm
- net +5V: track 24.4 -> 22.0 mm
- net EMER24V: track 23.0 -> 21.5 mm
- net ENTER: track 35.1 -> 35.7 mm
Other:
- board text added: "Autor: Antonio Pérez García Trabajo Fin de Grado. 2022"
- board text added: "Conexiones"
- board text removed: "MIC_B"
